File: esp32-flash.kicad_sch (KiCad schematic)
At the start: 2 parts, among them U10 W25Q32JVSIQ

Commit message: Cleanup WIP
Parts:
- renumbered C30 to C23, U10 to U8
Changed lines of the file:
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@@
 		(on_board yes)
 		(dnp no)
-		(property "Reference" "U10"
+		(property "Reference" "U8"
 			(at 156.21 88.265 0)
 			(effects
@@
 			(project "protea32"
 				(path "/8c0b3d8b-46d3-4173-ab1e-a61765f77d61/542878b0-9aae-45cf-ad58-4d9e0bda3cee/3907d691-16c9-46b9-8e1c-0399c2dec8f4"
-					(reference "U10")
+					(reference "U8")
 					(unit 1)
 				)
@@
 		(on_board yes)
 		(dnp no)
-		(property "Reference" "#PWR074"
+		(property "Reference" "#PWR054"
 			(at 162.56 119.38 0)
 			(effects
@@
 			(project "protea32"
 				(path "/8c0b3d8b-46d3-4173-ab1e-a61765f77d61/542878b0-9aae-45cf-ad58-4d9e0bda3cee/3907d691-16c9-46b9-8e1c-0399c2dec8f4"
-					(reference "#PWR074")
+					(reference "#PWR054")
 					(unit 1)
 				)
@@
 		(on_board yes)
 		(dnp no)
-		(property "Reference" "C30"
+		(property "Reference" "C23"
 			(at 177.038 80.264 90)
 			(effects
@@
 			)
 		)
-		(property "Datasheet" "https://eu.mouser.com/datasheet/2/40/KGM_X7R-3223212.pdf"
-			(at 175.26 83.82 0)
-			(effects
-				(font
-					(size 1.27 1.27)
-				)
-				(hide yes)
-			)
-		)
-		(property "Description" ""
+		(property "Datasheet" "~"
+			(at 175.26 83.82 0)
+			(effects
+				(font
+					(size 1.27 1.27)
+				)
+				(hide yes)
+			)
+		)
+		(property "Description" "Unpolarized capacitor"
 			(at 175.26 83.82 0)
 			(effects
@@
 			(project "protea32"
 				(path "/8c0b3d8b-46d3-4173-ab1e-a61765f77d61/542878b0-9aae-45cf-ad58-4d9e0bda3cee/3907d691-16c9-46b9-8e1c-0399c2dec8f4"
-					(reference "C30")
+					(reference "C23")
 					(unit 1)
 				)
@@
 		(on_board yes)
 		(dnp no)
-		(property "Reference" "#PWR075"
+		(property "Reference" "#PWR055"
 			(at 185.42 83.82 0)
 			(effects
@@
 			(project "protea32"
 				(path "/8c0b3d8b-46d3-4173-ab1e-a61765f77d61/542878b0-9aae-45cf-ad58-4d9e0bda3cee/3907d691-16c9-46b9-8e1c-0399c2dec8f4"
-					(reference "#PWR075")
-					(unit 1)
-				)
+					(reference "#PWR055")
+					(unit 1)
+				)
