File: esp32-psram.kicad_sch (KiCad schematic)
At the start: 3 parts, among them U13 ESP-PSRAM32

Commit message: Cleanup WIP
Parts:
- renumbered C52 to C45, R44 to R38, U13 to U12
Changed lines of the file:
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@@
 		(on_board yes)
 		(dnp no)
-		(property "Reference" "#PWR0147"
+		(property "Reference" "#PWR0127"
 			(at 170.18 114.3 0)
 			(effects
@@
 			(project "protea32"
 				(path "/8c0b3d8b-46d3-4173-ab1e-a61765f77d61/542878b0-9aae-45cf-ad58-4d9e0bda3cee/40a93926-f68e-4b17-bd29-d89ea6b5eee8"
-					(reference "#PWR0147")
+					(reference "#PWR0127")
 					(unit 1)
 				)
@@
 		(on_board yes)
 		(dnp no)
-		(property "Reference" "R44"
+		(property "Reference" "R38"
 			(at 153.8478 81.28 90)
 			(effects
@@
 			)
 		)
-		(property "Datasheet" "https://www.vishay.com/docs/28952/mcs0402at-mct0603at-mcu0805at-mca1206at.pdf"
+		(property "Datasheet" "~"
 			(at 148.59 81.28 0)
 			(effects
@@
 			)
 		)
-		(property "Description" ""
+		(property "Description" "Resistor"
 			(at 148.59 81.28 0)
 			(effects
@@
 			(project "protea32"
 				(path "/8c0b3d8b-46d3-4173-ab1e-a61765f77d61/542878b0-9aae-45cf-ad58-4d9e0bda3cee/40a93926-f68e-4b17-bd29-d89ea6b5eee8"
-					(reference "R44")
+					(reference "R38")
 					(unit 1)
 				)
@@
 		(on_board yes)
 		(dnp no)
-		(property "Reference" "#PWR0148"
+		(property "Reference" "#PWR0128"
 			(at 190.5 78.74 0)
 			(effects
@@
 			(project "protea32"
 				(path "/8c0b3d8b-46d3-4173-ab1e-a61765f77d61/542878b0-9aae-45cf-ad58-4d9e0bda3cee/40a93926-f68e-4b17-bd29-d89ea6b5eee8"
-					(reference "#PWR0148")
+					(reference "#PWR0128")
 					(unit 1)
 				)
@@
 		(on_board yes)
 		(dnp no)
-		(property "Reference" "U13"
+		(property "Reference" "U12"
 			(at 176.53 93.9799 0)
 			(effects
@@
 			(project "protea32"
 				(path "/8c0b3d8b-46d3-4173-ab1e-a61765f77d61/542878b0-9aae-45cf-ad58-4d9e0bda3cee/40a93926-f68e-4b17-bd29-d89ea6b5eee8"
-					(reference "U13")
+					(reference "U12")
 					(unit 1)
 				)
@@
 		(on_board yes)
 		(dnp no)
-		(property "Reference" "C52"
+		(property "Reference" "C45"
 			(at 182.118 75.184 90)
 			(effects
@@
 			)
 		)
-		(property "Datasheet" "https://www.vishay.com/docs/45199/vjcommercialseries.pdf"
+		(property "Datasheet" "~"
 			(at 180.34 78.74 0)
 			(effects
@@
 			)
 		)
-		(property "Description" ""
+		(property "Description" "Unpolarized capacitor"
 			(at 180.34 78.74 0)
 			(effects
@@
 			(project "protea32"
 				(path "/8c0b3d8b-46d3-4173-ab1e-a61765f77d61/542878b0-9aae-45cf-ad58-4d9e0bda3cee/40a93926-f68e-4b17-bd29-d89ea6b5eee8"
-					(reference "C52")
-					(unit 1)
-				)
+					(reference "C45")
+					(unit 1)
+				)

Commit message: HW 1.01
Parts:
- renumbered C45 to C27, R38 to R31
Changed lines of the file:
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@@
 		(on_board yes)
 		(dnp no)
-		(property "Reference" "#PWR0127"
+		(property "Reference" "#PWR0102"
 			(at 170.18 114.3 0)
 			(effects
@@
 		(instances
 			(project "protea32"
-				(path "/8c0b3d8b-46d3-4173-ab1e-a61765f77d61/542878b0-9aae-45cf-ad58-4d9e0bda3cee/40a93926-f68e-4b17-bd29-d89ea6b5eee8"
-					(reference "#PWR0127")
+				(path "/8c0b3d8b-46d3-4173-ab1e-a61765f77d61/b7bb8eb4-1c1a-4a33-b2e9-225ce0ce3935/40a93926-f68e-4b17-bd29-d89ea6b5eee8"
+					(reference "#PWR0102")
 					(unit 1)
 				)
@@
 		(on_board yes)
 		(dnp no)
-		(property "Reference" "R38"
+		(property "Reference" "R31"
 			(at 153.8478 81.28 90)
 			(effects
@@
 		(instances
 			(project "protea32"
-				(path "/8c0b3d8b-46d3-4173-ab1e-a61765f77d61/542878b0-9aae-45cf-ad58-4d9e0bda3cee/40a93926-f68e-4b17-bd29-d89ea6b5eee8"
-					(reference "R38")
+				(path "/8c0b3d8b-46d3-4173-ab1e-a61765f77d61/b7bb8eb4-1c1a-4a33-b2e9-225ce0ce3935/40a93926-f68e-4b17-bd29-d89ea6b5eee8"
+					(reference "R31")
 					(unit 1)
 				)
@@
 		(on_board yes)
 		(dnp no)
-		(property "Reference" "#PWR0128"
+		(property "Reference" "#PWR0103"
 			(at 190.5 78.74 0)
 			(effects
@@
 		(instances
 			(project "protea32"
-				(path "/8c0b3d8b-46d3-4173-ab1e-a61765f77d61/542878b0-9aae-45cf-ad58-4d9e0bda3cee/40a93926-f68e-4b17-bd29-d89ea6b5eee8"
-					(reference "#PWR0128")
+				(path "/8c0b3d8b-46d3-4173-ab1e-a61765f77d61/b7bb8eb4-1c1a-4a33-b2e9-225ce0ce3935/40a93926-f68e-4b17-bd29-d89ea6b5eee8"
+					(reference "#PWR0103")
 					(unit 1)
 				)
@@
 		(instances
 			(project "protea32"
-				(path "/8c0b3d8b-46d3-4173-ab1e-a61765f77d61/542878b0-9aae-45cf-ad58-4d9e0bda3cee/40a93926-f68e-4b17-bd29-d89ea6b5eee8"
+				(path "/8c0b3d8b-46d3-4173-ab1e-a61765f77d61/b7bb8eb4-1c1a-4a33-b2e9-225ce0ce3935/40a93926-f68e-4b17-bd29-d89ea6b5eee8"
 					(reference "U12")
 					(unit 1)
@@
 		(on_board yes)
 		(dnp no)
-		(property "Reference" "C45"
+		(property "Reference" "C27"
 			(at 182.118 75.184 90)
 			(effects
@@
 		(instances
 			(project "protea32"
-				(path "/8c0b3d8b-46d3-4173-ab1e-a61765f77d61/542878b0-9aae-45cf-ad58-4d9e0bda3cee/40a93926-f68e-4b17-bd29-d89ea6b5eee8"
-					(reference "C45")
-					(unit 1)
-				)
+				(path "/8c0b3d8b-46d3-4173-ab1e-a61765f77d61/b7bb8eb4-1c1a-4a33-b2e9-225ce0ce3935/40a93926-f68e-4b17-bd29-d89ea6b5eee8"
+					(reference "C27")
+					(unit 1)
+				)
