File: esp8266.kicad_sch (KiCad schematic)
At the start: 19 parts, among them U1 W25Q16JVSSIQ, U2 ESP8266EX, Y1 26 MHz Passive

Commit message: HW 1.01
Parts:
- added R39: 4.7K, FRANK:Resistor (0603), symbol Protea:R_Small
- added U13: DS2401P+, FRANK:TSOC-6, symbol DS2401P+:DS2401P+
Connections:
- net +3V3: now also R39.1
- net GND: now also U13.1 (GND)
- net GPIO5: now also R39.2, U13.2 (DATA)
- no-connect marks 1 -> 5
Other:
- moved on the sheet: AE1, C1, C2, C3, C4, C5, C6, C7, L1, R1, R2, R3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
