File: protea32.kicad_pcb (KiCad board)
At the start: 2 copper layers, 70 x 70 mm, 146 parts, among them J1 USB4215-03-A, J12 DC3RX19JA2, J2 676430910, J3 TTL, J4 D-SUB 9 Male, J5 0475710001, J6 Defaults, J7 Flash, Q1 2N7000, Q2 2N7000, Q3 2N7000, Q4 2N7000, Q5 2N7000, Q6 UMH3N, U1 USBLC6-2SC6, U10 74HC4052D, U11 CMT-7525-80-SMT-TR, U13 CH340C, U14 ESP32-D0WD-V3, U2 TS3USB221RSER, U3 NCP1117 3.3, U4 USBLC6-2SC6, U5 RP2040, U6 W25Q16JVSSIQ, U7 MAX232CSE+, U8 W25Q32JVSIQ, U9 74HC4052D, Y1 ASE-12MHz, Y2 40MHz

Commit message: HW 1.01
Parts:
- C1, C10, C11, C12, C13, C14, C15, C16, C17, C18, C19, C2, C20, C21, C22, C24, C25, C26, C28, C29, C3, C4, C5, C6, C7, C8, C9: footprint FRANK:Capacitor (0603) -> FRANK:Capacitor (0603, S)
- R1, R10, R11, R12, R13, R14, R15, R16, R17, R18, R19, R2, R20, R21, R22, R23, R24, R25, R26, R27, R28, R29, R3, R30, R32, R33, R4, R5, R6, R7, R8, R9: footprint FRANK:Resistor (0603) -> FRANK:Resistor (0603, S)
- moved LD3 14.8 mm to (164.0, 117.3), turned to 180 degrees
- moved U8 1.89 mm to (152.8, 109.3)
- moved C40 0.16 mm to (153.4, 116.1)
- moved C20 0.10 mm to (148.6, 93.7)
Routing:
- net Net-(LD3-A): track 3.54 -> 11.6 mm
- net /ESP_SDI/SD1: track 9.06 -> 5.63 mm
- net +3V3: track 237.1 -> 234.5 mm, vias 28 -> 30
- net /VDD_SDIO: track 13.1 -> 15.7 mm
- net /ESP_TXD: track 14.3 -> 16.4 mm
- net /ESP_SCK/CLK: track 9.29 -> 7.64 mm
- net /ESP_GPIO5: track 43.2 -> 44.6 mm
- net /ESP_SCS/CMD: track 15.7 -> 14.3 mm
- net /ESP_CHIP_PU: track 124.4 -> 125.5 mm
- net /ESP_U0TXD: track 19.3 -> 20.4 mm
- net /ESP_GPIO0: track 50.2 -> 51.1 mm
- net Net-(S1-B): track 53.1 -> 52.3 mm
- net /Multiplexers/MP_TX: track 17.1 -> 17.9 mm
- net GND: vias 47 -> 78
Other:
- outline, holes or cut-outs redrawn
- board text added: "32"
- board text added: "PROTEA"
- board text removed: "${NAME}"

Commit message: HW 1.01 Release
Parts:
- moved H3 3.61 mm to (126.9, 130.9)
- moved J4 3.00 mm to (131.6, 78.3)
- moved H1 3.00 mm to (126.9, 64.9)
- moved S4 3.00 mm to (125.4, 118.7)
- moved C26 2.90 mm to (171.3, 124.4), turned to -90 degrees
- moved C44 2.59 mm to (148.8, 126.8)
- moved AE1 2.46 mm to (146.6, 128.1)
- moved S1 2.13 mm to (184.1, 132.1)
- moved H4 2.00 mm to (193.9, 130.9)
- moved J5 1.98 mm to (171.9, 130.8)
- moved L2 1.22 mm to (146.6, 125.9), turned to 90 degrees
- moved C42 0.18 mm to (144.3, 125.0)
Routing:
- net VBUS: track 272.1 -> 276.4 mm
- net /RP_GPIO15: track 106.7 -> 110.8 mm
- net /ESP_CHIP_PU: track 125.5 -> 128.5 mm
- net /RS232, TTL/RX_IN: track 25.9 -> 28.9 mm
- net /RS232, TTL/TX_IN: track 30.7 -> 33.7 mm
- net /RS232, TTL/RTS_IN: track 32.6 -> 35.6 mm
- net /RS232, TTL/CTS_IN: track 32.3 -> 35.3 mm
- net +3V3: track 234.5 -> 237.2 mm
- net Net-(S1-B): track 52.3 -> 54.4 mm
- net /ESP_GPIO5: track 44.6 -> 46.6 mm
- net /ESP_GPIO23: track 39.7 -> 41.6 mm
- net /ESP_GPIO19: track 30.5 -> 32.4 mm
- net /ESP_GPIO18: track 34.8 -> 36.7 mm
- net GND: track 12.3 -> 13.8 mm, vias 78 -> 95
Other:
- board size 70 x 70 mm -> 73 x 72 mm
