File: protea32.kicad_sch (KiCad schematic)
At the start: 4 parts

Commit message: Cleanup WIP
Changed lines of the file:
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@@
 		)
 	)
-	(label "UT_RTS"
+	(label "ESP_RTS"
 		(at 27.94 116.84 0)
 		(effects
@@
 		)
 	)
-	(label "UT_DTR"
+	(label "ESP_DTR"
 		(at 27.94 114.3 0)
 		(effects

Commit message: HW 1.01
Connections:
- no-connect marks 32 -> 33
