File: buzzer.kicad_sch (KiCad schematic)
At the start: 5 parts, among them Q5 2N7000

Commit message: Cleanup WIP
Parts:
- renumbered R28 to R22, R29 to R23
Changed lines of the file:
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@@
 		(dnp no)
 		(fields_autoplaced yes)
-		(property "Reference" "#PWR099"
+		(property "Reference" "#PWR079"
 			(at 135.89 62.23 0)
 			(effects
@@
 			(project "protea"
 				(path "/8c0b3d8b-46d3-4173-ab1e-a61765f77d61/745a17db-43e3-4b47-bd96-a8d1c23cf5c8"
-					(reference "#PWR099")
+					(reference "#PWR079")
 					(unit 1)
 				)
@@
 		(dnp no)
 		(fields_autoplaced yes)
-		(property "Reference" "#PWR0100"
+		(property "Reference" "#PWR080"
 			(at 135.89 114.3 0)
 			(effects
@@
 			(project "protea"
 				(path "/8c0b3d8b-46d3-4173-ab1e-a61765f77d61/745a17db-43e3-4b47-bd96-a8d1c23cf5c8"
-					(reference "#PWR0100")
+					(reference "#PWR080")
 					(unit 1)
 				)
@@
 		(on_board yes)
 		(dnp no)
-		(property "Reference" "R29"
+		(property "Reference" "R23"
 			(at 122.428 91.694 90)
 			(effects
@@
 			(project "protea"
 				(path "/8c0b3d8b-46d3-4173-ab1e-a61765f77d61/745a17db-43e3-4b47-bd96-a8d1c23cf5c8"
-					(reference "R29")
+					(reference "R23")
 					(unit 1)
 				)
@@
 		(dnp no)
 		(fields_autoplaced yes)
-		(property "Reference" "#PWR098"
+		(property "Reference" "#PWR078"
 			(at 114.3 114.3 0)
 			(effects
@@
 			(project "protea"
 				(path "/8c0b3d8b-46d3-4173-ab1e-a61765f77d61/745a17db-43e3-4b47-bd96-a8d1c23cf5c8"
-					(reference "#PWR098")
+					(reference "#PWR078")
 					(unit 1)
 				)
@@
 		(on_board yes)
 		(dnp no)
-		(property "Reference" "R28"
+		(property "Reference" "R22"
 			(at 112.014 104.648 90)
 			(effects
@@
 			(project "protea"
 				(path "/8c0b3d8b-46d3-4173-ab1e-a61765f77d61/745a17db-43e3-4b47-bd96-a8d1c23cf5c8"
-					(reference "R28")
-					(unit 1)
-				)
+					(reference "R22")
+					(unit 1)
+				)

Commit message: HW 1.01
Parts:
- R22, R23: footprint FRANK:Resistor (0603, S) -> FRANK:Resistor (0603)
- renumbered LS1 to U11
Changed lines of the file:
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@@
 		(rev "${VERSION}")
 		(company "Mikhail Matveev")
-		(comment 1 "https://github.com/xtremespb/frank")
+		(comment 1 "https://github.com/rh1tech/protea")
 	)
 	(junction
@@
 			)
 		)
-		(property "Footprint" "FRANK:Resistor (0603, S)"
+		(property "Footprint" "FRANK:Resistor (0603)"
 			(at 120.65 92.202 90)
 			(effects
@@
 			)
 		)
-		(property "Footprint" "FRANK:Resistor (0603, S)"
+		(property "Footprint" "FRANK:Resistor (0603)"
 			(at 116.078 102.87 90)
 			(effects
@@
 		(dnp no)
 		(fields_autoplaced yes)
-		(property "Reference" "LS1"
+		(property "Reference" "U11"
 			(at 153.67 63.5 0)
 			(effects
@@
 			(project "protea"
 				(path "/8c0b3d8b-46d3-4173-ab1e-a61765f77d61/745a17db-43e3-4b47-bd96-a8d1c23cf5c8"
-					(reference "LS1")
+					(reference "U11")
 					(unit 1)
 				)

Commit message: HW 1.01
Parts:
- R22, R23: footprint FRANK:Resistor (0603) -> FRANK:Resistor (0603, S)
Changed lines of the file:
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@@
 			)
 		)
-		(property "Footprint" "FRANK:Resistor (0603)"
+		(property "Footprint" "FRANK:Resistor (0603, S)"
 			(at 120.65 92.202 90)
 			(effects
@@
 			)
 		)
-		(property "Footprint" "FRANK:Resistor (0603)"
+		(property "Footprint" "FRANK:Resistor (0603, S)"
 			(at 116.078 102.87 90)
 			(effects
