File: jumpers.kicad_sch (KiCad schematic)
At the start: 13 parts, among them J6 Flash

Commit message: Cleanup WIP
Parts:
- renumbered R33 to R27, R34 to R28, R35 to R29
Changed lines of the file:
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@@
 		(on_board yes)
 		(dnp no)
-		(property "Reference" "#PWR0111"
+		(property "Reference" "#PWR091"
 			(at 110.49 101.6 0)
 			(effects
@@
 			(project "protea"
 				(path "/8c0b3d8b-46d3-4173-ab1e-a61765f77d61/6a818bab-ab6c-4357-bafe-0bf3a24e9049"
-					(reference "#PWR0111")
+					(reference "#PWR091")
 					(unit 1)
 				)
@@
 		(dnp no)
 		(fields_autoplaced yes)
-		(property "Reference" "#PWR0115"
+		(property "Reference" "#PWR095"
 			(at 170.18 67.31 0)
 			(effects
@@
 			(project "protea"
 				(path "/8c0b3d8b-46d3-4173-ab1e-a61765f77d61/6a818bab-ab6c-4357-bafe-0bf3a24e9049"
-					(reference "#PWR0115")
+					(reference "#PWR095")
 					(unit 1)
 				)
@@
 		(dnp no)
 		(fields_autoplaced yes)
-		(property "Reference" "#PWR0112"
+		(property "Reference" "#PWR092"
 			(at 120.65 104.14 0)
 			(effects
@@
 			(project "protea"
 				(path "/8c0b3d8b-46d3-4173-ab1e-a61765f77d61/6a818bab-ab6c-4357-bafe-0bf3a24e9049"
-					(reference "#PWR0112")
+					(reference "#PWR092")
 					(unit 1)
 				)
@@
 		(on_board yes)
 		(dnp no)
-		(property "Reference" "#PWR0119"
+		(property "Reference" "#PWR099"
 			(at 193.04 109.22 0)
 			(effects
@@
 			(project "protea"
 				(path "/8c0b3d8b-46d3-4173-ab1e-a61765f77d61/6a818bab-ab6c-4357-bafe-0bf3a24e9049"
-					(reference "#PWR0119")
+					(reference "#PWR099")
 					(unit 1)
 				)
@@
 		(dnp no)
 		(fields_autoplaced yes)
-		(property "Reference" "R35"
+		(property "Reference" "R29"
 			(at 187.96 60.96 90)
 			(effects
@@
 			(project "protea"
 				(path "/8c0b3d8b-46d3-4173-ab1e-a61765f77d61/6a818bab-ab6c-4357-bafe-0bf3a24e9049"
-					(reference "R35")
+					(reference "R29")
 					(unit 1)
 				)
@@
 		(on_board yes)
 		(dnp no)
-		(property "Reference" "#PWR0117"
+		(property "Reference" "#PWR097"
 			(at 203.2 77.47 0)
 			(effects
@@
 			(project "protea"
 				(path "/8c0b3d8b-46d3-4173-ab1e-a61765f77d61/6a818bab-ab6c-4357-bafe-0bf3a24e9049"
-					(reference "#PWR0117")
+					(reference "#PWR097")
 					(unit 1)
 				)
@@
 		(on_board yes)
 		(dnp no)
-		(property "Reference" "R34"
+		(property "Reference" "R28"
 			(at 184.15 75.438 90)
 			(effects
@@
 			(project "protea"
 				(path "/8c0b3d8b-46d3-4173-ab1e-a61765f77d61/6a818bab-ab6c-4357-bafe-0bf3a24e9049"
-					(reference "R34")
+					(reference "R28")
 					(unit 1)
 				)
@@
 		(on_board yes)
 		(dnp no)
-		(property "Reference" "#PWR0113"
+		(property "Reference" "#PWR093"
 			(at 110.49 113.03 0)
 			(effects
@@
 			(project "protea"
 				(path "/8c0b3d8b-46d3-4173-ab1e-a61765f77d61/6a818bab-ab6c-4357-bafe-0bf3a24e9049"
-					(reference "#PWR0113")
+					(reference "#PWR093")
 					(unit 1)
 				)
@@
 		(on_board yes)
 		(dnp no)
-		(property "Reference" "#PWR0118"
+		(property "Reference" "#PWR098"
 			(at 203.2 106.68 0)
 			(effects
@@
 			(project "protea"
 				(path "/8c0b3d8b-46d3-4173-ab1e-a61765f77d61/6a818bab-ab6c-4357-bafe-0bf3a24e9049"
-					(reference "#PWR0118")
+					(reference "#PWR098")
 					(unit 1)
 				)
@@
 		(dnp no)
 		(fields_autoplaced yes)
-		(property "Reference" "#PWR0114"
+		(property "Reference" "#PWR094"
 			(at 120.65 115.57 0)
 			(effects
@@
 			(project "protea"
 				(path "/8c0b3d8b-46d3-4173-ab1e-a61765f77d61/6a818bab-ab6c-4357-bafe-0bf3a24e9049"
-					(reference "#PWR0114")
+					(reference "#PWR094")
 					(unit 1)
 				)
@@
 		(on_board yes)
 		(dnp no)
-		(property "Reference" "#PWR0110"
+		(property "Reference" "#PWR090"
 			(at 109.22 140.97 0)
 			(effects
@@
 			(project "protea"
 				(path "/8c0b3d8b-46d3-4173-ab1e-a61765f77d61/6a818bab-ab6c-4357-bafe-0bf3a24e9049"
-					(reference "#PWR0110")
+					(reference "#PWR090")
 					(unit 1)
 				)
@@
 		(dnp no)
 		(fields_autoplaced yes)
-		(property "Reference" "#PWR0116"
+		(property "Reference" "#PWR096"
 			(at 190.5 67.31 0)
 			(effects
@@
 			(project "protea"
 				(path "/8c0b3d8b-46d3-4173-ab1e-a61765f77d61/6a818bab-ab6c-4357-bafe-0bf3a24e9049"
-					(reference "#PWR0116")
+					(reference "#PWR096")
 					(unit 1)
 				)
@@
 		(on_board yes)
 		(dnp no)
-		(property "Reference" "R33"
+		(property "Reference" "R27"
 			(at 124.46 124.206 90)
 			(effects
@@
 			(project "protea"
 				(path "/8c0b3d8b-46d3-4173-ab1e-a61765f77d61/6a818bab-ab6c-4357-bafe-0bf3a24e9049"
-					(reference "R33")
+					(reference "R27")
 					(unit 1)
 				)
@@
 		(on_board yes)
 		(dnp no)
-		(property "Reference" "#PWR0120"
+		(property "Reference" "#PWR0100"
 			(at 193.04 111.76 0)
 			(effects
@@
 			(project "protea"
 				(path "/8c0b3d8b-46d3-4173-ab1e-a61765f77d61/6a818bab-ab6c-4357-bafe-0bf3a24e9049"
-					(reference "#PWR0120")
-					(unit 1)
-				)
+					(reference "#PWR0100")
+					(unit 1)
+				)

Commit message: HW 1.01
Parts:
- added S4: ESP RST, FRANK:TACT-SIDE-4623, symbol Protea:SW_Push
- J7: renamed from J6; footprint FRANK:TACT-SIDE-4623 -> FRANK:Button (SMD, 3x3mm, 1-1)
- R28: renamed from R27; footprint FRANK:Resistor (0603, S) -> FRANK:Resistor (0603)
- R29: renamed from R28; footprint FRANK:Resistor (0603, S) -> FRANK:Resistor (0603)
- R30: renamed from R29; footprint FRANK:Resistor (0603, S) -> FRANK:Resistor (0603)
- renumbered J9 to J10, J10 to J11, TP1 to J6, J7 to J8, J8 to J9
Connections:
- net ESP_RESET: now also S4.1
- net GND: now also S4.2

Commit message: HW 1.01
Parts:
- R28, R29, R30: footprint FRANK:Resistor (0603) -> FRANK:Resistor (0603, S)
Changed lines of the file:
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@@
 			)
 		)
-		(property "Footprint" "FRANK:Resistor (0603)"
+		(property "Footprint" "FRANK:Resistor (0603, S)"
 			(at 187.96 69.088 90)
 			(effects
@@
 			)
 		)
-		(property "Footprint" "FRANK:Resistor (0603)"
+		(property "Footprint" "FRANK:Resistor (0603, S)"
 			(at 184.15 77.47 0)
 			(effects
@@
 			)
 		)
-		(property "Footprint" "FRANK:Resistor (0603)"
+		(property "Footprint" "FRANK:Resistor (0603, S)"
 			(at 124.46 127 0)
 			(effects
