File: power.kicad_sch (KiCad schematic)
At the start: 20 parts, among them J1 USB4215-03-A, J2 676430910, U3 USBLC6-2SC6, U4 TS3USB221RSER, U5 NCP1117 3.3, U6 USBLC6-2SC6

Commit message: Cleanup WIP
Parts:
- renumbered C8 to C1, C9 to C2, C10 to C3, C11 to C4, R7 to R1, R8 to R2, R9 to R3, R10 to R4, R11 to R5, R12 to R6, R13 to R7, R14 to R8, R15 to R9, S2 to S1, U3 to U1, U4 to U2, U5 to U3, U6 to U4

Commit message: HW 1.01
Parts:
- C1, C2, C3, C4: footprint FRANK:Capacitor (0603, S) -> FRANK:Capacitor (0603)
- R1, R2, R3, R4, R5, R6, R7, R8, R9: footprint FRANK:Resistor (0603, S) -> FRANK:Resistor (0603)
Changed lines of the file:
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@@
 		(rev "${VERSION}")
 		(company "Mikhail Matveev")
-		(comment 1 "https://github.com/xtremespb/frank")
+		(comment 1 "https://github.com/rh1tech/protea")
 	)
 	(junction
@@
 			)
 		)
-		(property "Footprint" "FRANK:Capacitor (0603, S)"
+		(property "Footprint" "FRANK:Capacitor (0603)"
 			(at 200.3552 97.79 0)
 			(effects
@@
 			)
 		)
-		(property "Footprint" "FRANK:Resistor (0603, S)"
+		(property "Footprint" "FRANK:Resistor (0603)"
 			(at 106.172 128.27 90)
 			(effects
@@
 			)
 		)
-		(property "Footprint" "FRANK:Capacitor (0603, S)"
+		(property "Footprint" "FRANK:Capacitor (0603)"
 			(at 163.5252 99.06 0)
 			(effects
@@
 			)
 		)
-		(property "Footprint" "FRANK:Resistor (0603, S)"
+		(property "Footprint" "FRANK:Resistor (0603)"
 			(at 104.14 96.52 0)
 			(effects
@@
 			)
 		)
-		(property "Footprint" "FRANK:Resistor (0603, S)"
+		(property "Footprint" "FRANK:Resistor (0603)"
 			(at 146.812 165.1 90)
 			(effects
@@
 			)
 		)
-		(property "Footprint" "FRANK:Resistor (0603, S)"
+		(property "Footprint" "FRANK:Resistor (0603)"
 			(at 120.142 54.61 90)
 			(effects
@@
 			)
 		)
-		(property "Footprint" "FRANK:Resistor (0603, S)"
+		(property "Footprint" "FRANK:Resistor (0603)"
 			(at 185.42 146.558 90)
 			(effects
@@
 			)
 		)
-		(property "Footprint" "FRANK:Capacitor (0603, S)"
+		(property "Footprint" "FRANK:Capacitor (0603)"
 			(at 164.1348 130.81 0)
 			(effects
@@
 			)
 		)
-		(property "Footprint" "FRANK:Resistor (0603, S)"
+		(property "Footprint" "FRANK:Resistor (0603)"
 			(at 125.73 105.918 90)
 			(effects
@@
 			)
 		)
-		(property "Footprint" "FRANK:Resistor (0603, S)"
+		(property "Footprint" "FRANK:Resistor (0603)"
 			(at 125.73 108.458 90)
 			(effects
@@
 			)
 		)
-		(property "Footprint" "FRANK:Resistor (0603, S)"
+		(property "Footprint" "FRANK:Resistor (0603)"
 			(at 104.14 111.76 0)
 			(effects
@@
 			)
 		)
-		(property "Footprint" "FRANK:Resistor (0603, S)"
+		(property "Footprint" "FRANK:Resistor (0603)"
 			(at 185.42 149.098 90)
 			(effects
@@
 			)
 		)
-		(property "Footprint" "FRANK:Capacitor (0603, S)"
+		(property "Footprint" "FRANK:Capacitor (0603)"
 			(at 147.32 39.6748 0)
 			(effects

Commit message: HW 1.01
Parts:
- C1, C2, C3, C4: footprint FRANK:Capacitor (0603) -> FRANK:Capacitor (0603, S)
- R1, R2, R3, R4, R5, R6, R7, R8, R9: footprint FRANK:Resistor (0603) -> FRANK:Resistor (0603, S)
Changed lines of the file:
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@@
 			)
 		)
-		(property "Footprint" "FRANK:Capacitor (0603)"
+		(property "Footprint" "FRANK:Capacitor (0603, S)"
 			(at 200.3552 97.79 0)
 			(effects
@@
 			)
 		)
-		(property "Footprint" "FRANK:Resistor (0603)"
+		(property "Footprint" "FRANK:Resistor (0603, S)"
 			(at 106.172 128.27 90)
 			(effects
@@
 			)
 		)
-		(property "Footprint" "FRANK:Capacitor (0603)"
+		(property "Footprint" "FRANK:Capacitor (0603, S)"
 			(at 163.5252 99.06 0)
 			(effects
@@
 			)
 		)
-		(property "Footprint" "FRANK:Resistor (0603)"
+		(property "Footprint" "FRANK:Resistor (0603, S)"
 			(at 104.14 96.52 0)
 			(effects
@@
 			)
 		)
-		(property "Footprint" "FRANK:Resistor (0603)"
+		(property "Footprint" "FRANK:Resistor (0603, S)"
 			(at 146.812 165.1 90)
 			(effects
@@
 			)
 		)
-		(property "Footprint" "FRANK:Resistor (0603)"
+		(property "Footprint" "FRANK:Resistor (0603, S)"
 			(at 120.142 54.61 90)
 			(effects
@@
 			)
 		)
-		(property "Footprint" "FRANK:Resistor (0603)"
+		(property "Footprint" "FRANK:Resistor (0603, S)"
 			(at 185.42 146.558 90)
 			(effects
@@
 			)
 		)
-		(property "Footprint" "FRANK:Capacitor (0603)"
+		(property "Footprint" "FRANK:Capacitor (0603, S)"
 			(at 164.1348 130.81 0)
 			(effects
@@
 			)
 		)
-		(property "Footprint" "FRANK:Resistor (0603)"
+		(property "Footprint" "FRANK:Resistor (0603, S)"
 			(at 125.73 105.918 90)
 			(effects
@@
 			)
 		)
-		(property "Footprint" "FRANK:Resistor (0603)"
+		(property "Footprint" "FRANK:Resistor (0603, S)"
 			(at 125.73 108.458 90)
 			(effects
@@
 			)
 		)
-		(property "Footprint" "FRANK:Resistor (0603)"
+		(property "Footprint" "FRANK:Resistor (0603, S)"
 			(at 104.14 111.76 0)
 			(effects
@@
 			)
 		)
-		(property "Footprint" "FRANK:Resistor (0603)"
+		(property "Footprint" "FRANK:Resistor (0603, S)"
 			(at 185.42 149.098 90)
 			(effects
@@
 			)
 		)
-		(property "Footprint" "FRANK:Capacitor (0603)"
+		(property "Footprint" "FRANK:Capacitor (0603, S)"
 			(at 147.32 39.6748 0)
 			(effects
