File: rp2040.kicad_sch (KiCad schematic)
At the start: 24 parts, among them U7 RP2040, U8 W25Q16JVSSIQ, Y2 ASE-12MHz

Commit message: Cleanup WIP
Parts:
- renumbered C17 to C10, C18 to C11, C19 to C12, C20 to C13, C21 to C14, C22 to C15, C23 to C16, C24 to C17, C25 to C18, C12 to C5, C13 to C6, C14 to C7, C15 to C8, C16 to C9, R16 to R10, R17 to R11, R18 to R12, R19 to R13, S3 to S2, S4 to S3, U7 to U5, U8 to U6, Y2 to Y1

Commit message: HW 1.01
Parts:
- C10, C11, C12, C13, C14, C15, C16, C17, C18, C5, C6, C7, C8, C9: footprint FRANK:Capacitor (0603, S) -> FRANK:Capacitor (0603)
- R10, R11, R12, R13: footprint FRANK:Resistor (0603, S) -> FRANK:Resistor (0603)
Other:
- moved on the sheet: LD1, R13, S3
Changed lines of the file:
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@@
 		(rev "${VERSION}")
 		(company "Mikhail Matveev")
-		(comment 1 "https://github.com/xtremespb/frank")
+		(comment 1 "https://github.com/rh1tech/protea")
 	)
 	(text "Close to 44"
@@
 	(wire
 		(pts
-			(xy 264.16 130.81) (xy 266.7 130.81)
+			(xy 250.19 129.54) (xy 252.73 129.54)
 		)
 		(stroke
@@
 	(wire
 		(pts
-			(xy 261.62 144.78) (xy 271.78 144.78)
+			(xy 247.65 143.51) (xy 257.81 143.51)
 		)
 		(stroke
@@
 	)
 	(label "RUN"
-		(at 271.78 144.78 180)
+		(at 257.81 143.51 180)
 		(effects
 			(font
@@
 	)
 	(label "GPIO25"
-		(at 266.7 130.81 0)
+		(at 252.73 129.54 0)
 		(effects
 			(font
@@
 			)
 		)
-		(property "Footprint" "FRANK:Capacitor (0603, S)"
+		(property "Footprint" "FRANK:Capacitor (0603)"
 			(at 47.9552 46.99 0)
 			(effects
@@
 	(symbol
 		(lib_id "Protea:R")
-		(at 260.35 130.81 90)
+		(at 246.38 129.54 90)
 		(unit 1)
 		(exclude_from_sim no)
@@
 		(fields_autoplaced yes)
 		(property "Reference" "R13"
-			(at 260.35 124.46 90)
+			(at 246.38 123.19 90)
 			(effects
 				(font
@@
 		)
 		(property "Value" "1K"
-			(at 260.35 127 90)
+			(at 246.38 125.73 90)
 			(effects
 				(font
@@
 			)
 		)
-		(property "Footprint" "FRANK:Resistor (0603, S)"
-			(at 260.35 132.588 90)
+		(property "Footprint" "FRANK:Resistor (0603)"
+			(at 246.38 131.318 90)
 			(effects
 				(font
@@
 		)
 		(property "Datasheet" "https://www.vishay.com/docs/28952/mcs0402at-mct0603at-mcu0805at-mca1206at.pdf"
-			(at 260.35 130.81 0)
+			(at 246.38 129.54 0)
 			(effects
 				(font
@@
 		)
 		(property "Description" "Resistor"
-			(at 260.35 130.81 0)
+			(at 246.38 129.54 0)
 			(effects
 				(font
@@
 		)
 		(property "AliExpress" "https://www.aliexpress.com/item/1005005945735199.html"
-			(at 260.35 130.81 0)
+			(at 246.38 129.54 0)
 			(effects
 				(font
@@
 		)
 		(property "MANUFACTURER" ""
-			(at 260.35 130.81 0)
+			(at 246.38 129.54 0)
 			(effects
 				(font
@@
 			)
 		)
-		(property "Footprint" "FRANK:Capacitor (0603, S)"
+		(property "Footprint" "FRANK:Capacitor (0603)"
 			(at 136.8552 46.99 0)
 			(effects
@@
 	(symbol
 		(lib_id "Protea:GND")
-		(at 248.92 130.81 270)
+		(at 234.95 129.54 270)
 		(unit 1)
 		(exclude_from_sim no)
@@
 		(dnp no)
 		(fields_autoplaced yes)
-		(property "Reference" "#PWR035"
-			(at 242.57 130.81 0)
+		(property "Reference" "#PWR034"
+			(at 228.6 129.54 0)
 			(effects
 				(font
@@
 		)
 		(property "Value" "GND"
-			(at 245.11 130.8099 90)
+			(at 231.14 129.5399 90)
 			(effects
 				(font
@@
 		)
 		(property "Footprint" ""
-			(at 248.92 130.81 0)
+			(at 234.95 129.54 0)
 			(effects
 				(font
@@
 		)
 		(property "Datasheet" ""
-			(at 248.92 130.81 0)
+			(at 234.95 129.54 0)
 			(effects
 				(font
@@
 		)
 		(property "Description" "Power symbol creates a global label with name \"GND\" , ground"
-			(at 248.92 130.81 0)
+			(at 234.95 129.54 0)
 			(effects
 				(font
@@
 			(project "frank2"
 				(path "/8c0b3d8b-46d3-4173-ab1e-a61765f77d61/4beb664e-83a7-44f7-9571-ceb4c4bcb1db"
-					(reference "#PWR035")
+					(reference "#PWR034")
 					(unit 1)
 				)
@@
 			)
 		)
-		(property "Footprint" "FRANK:Resistor (0603, S)"
+		(property "Footprint" "FRANK:Resistor (0603)"
 			(at 123.19 79.502 90)
 			(effects
@@
 			)
 		)
-		(property "Footprint" "FRANK:Resistor (0603, S)"
+		(property "Footprint" "FRANK:Resistor (0603)"
 			(at 123.19 71.882 90)
 			(effects
@@
 	(symbol
 		(lib_id "Protea:GND")
-		(at 251.46 144.78 270)
+		(at 237.49 143.51 270)
 		(unit 1)
 		(exclude_from_sim no)
@@
 		(dnp no)
 		(fields_autoplaced yes)
-		(property "Reference" "#PWR037"
-			(at 245.11 144.78 0)
+		(property "Reference" "#PWR036"
+			(at 231.14 143.51 0)
 			(effects
 				(font
@@
 		)
 		(property "Value" "GND"
-			(at 247.65 144.7799 90)
+			(at 233.68 143.5099 90)
 			(effects
 				(font
@@
 		)
 		(property "Footprint" ""
-			(at 251.46 144.78 0)
+			(at 237.49 143.51 0)
 			(effects
 				(font
@@
 		)
 		(property "Datasheet" ""
-			(at 251.46 144.78 0)
+			(at 237.49 143.51 0)
 			(effects
 				(font
@@
 		)
 		(property "Description" "Power symbol creates a global label with name \"GND\" , ground"
-			(at 251.46 144.78 0)
+			(at 237.49 143.51 0)
 			(effects
 				(font
@@
 			(project "protea"
 				(path "/8c0b3d8b-46d3-4173-ab1e-a61765f77d61/4beb664e-83a7-44f7-9571-ceb4c4bcb1db"
-					(reference "#PWR037")
+					(reference "#PWR036")
 					(unit 1)
 				)
@@
 			)
 		)
-		(property "Footprint" "FRANK:Capacitor (0603, S)"
+		(property "Footprint" "FRANK:Capacitor (0603)"
 			(at 36.5252 46.99 0)
 			(effects
@@
 		(on_board yes)
 		(dnp no)
-		(property "Reference" "#PWR034"
+		(property "Reference" "#PWR035"
 			(at 236.22 104.14 0)
 			(effects
@@
 			(project "frank2"
 				(path "/8c0b3d8b-46d3-4173-ab1e-a61765f77d61/4beb664e-83a7-44f7-9571-ceb4c4bcb1db"
-					(reference "#PWR034")
+					(reference "#PWR035")
 					(unit 1)
 				)
@@
 			)
 		)
-		(property "Footprint" "FRANK:Capacitor (0603, S)"
+		(property "Footprint" "FRANK:Capacitor (0603)"
 			(at 164.7952 125.73 0)
 			(effects
@@
 			)
 		)
-		(property "Footprint" "FRANK:Capacitor (0603, S)"
+		(property "Footprint" "FRANK:Capacitor (0603)"
 			(at 102.5652 46.99 0)
 			(effects
@@
 		(on_board yes)
 		(dnp no)
-		(property "Reference" "#PWR036"
+		(property "Reference" "#PWR037"
 			(at 245.11 76.2 0)
 			(effects
@@
 			(project "frank2"
 				(path "/8c0b3d8b-46d3-4173-ab1e-a61765f77d61/4beb664e-83a7-44f7-9571-ceb4c4bcb1db"
-					(reference "#PWR036")
+					(reference "#PWR037")
 					(unit 1)
 				)
@@
 			)
 		)
-		(property "Footprint" "FRANK:Capacitor (0603, S)"
+		(property "Footprint" "FRANK:Capacitor (0603)"
 			(at 113.9952 46.99 0)
 			(effects
@@
 			)
 		)
-		(property "Footprint" "FRANK:Capacitor (0603, S)"
+		(property "Footprint" "FRANK:Capacitor (0603)"
 			(at 102.5652 62.23 0)
 			(effects
@@
 			)
 		)
-		(property "Footprint" "FRANK:Capacitor (0603, S)"
+		(property "Footprint" "FRANK:Capacitor (0603)"
 			(at 252.73 77.1652 0)
 			(effects
@@
 	(symbol
 		(lib_id "Protea:SW_Push")
-		(at 256.54 144.78 180)
+		(at 242.57 143.51 180)
 		(unit 1)
 		(exclude_from_sim no)
@@
 		(fields_autoplaced yes)
 		(property "Reference" "S3"
-			(at 256.54 139.7 0)
+			(at 242.57 138.43 0)
 			(effects
 				(font
@@
 		)
 		(property "Value" "Reset"
-			(at 256.54 142.24 0)
+			(at 242.57 140.97 0)
 			(effects
 				(font
@@
 		)
 		(property "Footprint" "FRANK:TACT-SIDE-4623"
-			(at 256.54 149.86 0)
+			(at 242.57 148.59 0)
 			(effects
 				(font
@@
 		)
 		(property "Datasheet" "https://parts4laptops.eu/en/microbuttons/3300-microbutton-tact-switch-ts-1233-33x33x15mm-smt-mounting.html"
-			(at 256.54 149.86 0)
+			(at 242.57 148.59 0)
 			(effects
 				(font
@@
 		)
 		(property "Description" ""
-			(at 256.54 144.78 0)
+			(at 242.57 143.51 0)
 			(effects
 				(font
@@
 		)
 		(property "AliExpress" "https://www.aliexpress.com/item/1005007359248990.html"
-			(at 256.54 144.78 0)
+			(at 242.57 143.51 0)
 			(effects
 				(font
@@
 		)
 		(property "Sim.Device" ""
-			(at 256.54 144.78 0)
+			(at 242.57 143.51 0)
 			(effects
 				(font
@@
 		)
 		(property "MANUFACTURER" ""
-			(at 256.54 144.78 0)
+			(at 242.57 143.51 0)
 			(effects
 				(font
@@
 			)
 		)
-		(property "Footprint" "FRANK:Capacitor (0603, S)"
+		(property "Footprint" "FRANK:Capacitor (0603)"
 			(at 182.5752 46.99 0)
 			(effects
@@
 	(symbol
 		(lib_id "Protea:LED")
-		(at 252.73 130.81 0)
+		(at 238.76 129.54 0)
 		(unit 1)
 		(exclude_from_sim no)
@@
 		(fields_autoplaced yes)
 		(property "Reference" "LD1"
-			(at 251.1425 124.46 0)
+			(at 237.1725 123.19 0)
 			(effects
 				(font
@@
 		)
 		(property "Value" "Blue"
-			(at 251.1425 127 0)
+			(at 237.1725 125.73 0)
 			(effects
 				(font
@@
 		)
 		(property "Footprint" "FRANK:LED (0805)"
-			(at 252.73 130.81 0)
+			(at 238.76 129.54 0)
 			(effects
 				(font
@@
 		)
 		(property "Datasheet" "https://www.farnell.com/datasheets/1760130.pdf"
-			(at 252.73 130.81 0)
+			(at 238.76 129.54 0)
 			(effects
 				(font
@@
 		)
 		(property "Description" "Light emitting diode"
-			(at 252.73 130.81 0)
+			(at 238.76 129.54 0)
 			(effects
 				(font
@@
 		)
 		(property "AliExpress" "https://www.aliexpress.com/item/1005007252088951.html"
-			(at 252.73 130.81 0)
+			(at 238.76 129.54 0)
 			(effects
 				(font
@@
 		)
 		(property "Sim.Pins" "1=K 2=A"
-			(at 252.73 130.81 0)
+			(at 238.76 129.54 0)
 			(effects
 				(font
@@
 		)
 		(property "MANUFACTURER" ""
-			(at 252.73 130.81 0)
+			(at 238.76 129.54 0)
 			(effects
 				(font
@@
 			)
 		)
-		(property "Footprint" "FRANK:Capacitor (0603, S)"
+		(property "Footprint" "FRANK:Capacitor (0603)"
 			(at 47.9552 62.23 0)
 			(effects
@@
 			)
 		)
-		(property "Footprint" "FRANK:Capacitor (0603, S)"
+		(property "Footprint" "FRANK:Capacitor (0603)"
 			(at 125.4252 46.99 0)
 			(effects
@@
 			)
 		)
-		(property "Footprint" "FRANK:Capacitor (0603, S)"
+		(property "Footprint" "FRANK:Capacitor (0603)"
 			(at 171.1452 46.99 0)
 			(effects
@@
 			)
 		)
-		(property "Footprint" "FRANK:Resistor (0603, S)"
+		(property "Footprint" "FRANK:Resistor (0603)"
 			(at 198.12 75.692 90)
 			(effects
@@
 			)
 		)
-		(property "Footprint" "FRANK:Capacitor (0603, S)"
+		(property "Footprint" "FRANK:Capacitor (0603)"
 			(at 148.2852 46.99 0)
 			(effects
@@
 			)
 		)
-		(property "Footprint" "FRANK:Capacitor (0603, S)"
+		(property "Footprint" "FRANK:Capacitor (0603)"
 			(at 159.7152 46.99 0)
 			(effects

Commit message: HW 1.01
Parts:
- C10, C11, C12, C13, C14, C15, C16, C17, C18, C5, C6, C7, C8, C9: footprint FRANK:Capacitor (0603) -> FRANK:Capacitor (0603, S)
- R10, R11, R12, R13: footprint FRANK:Resistor (0603) -> FRANK:Resistor (0603, S)
Changed lines of the file:
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@@
 			)
 		)
-		(property "Footprint" "FRANK:Capacitor (0603)"
+		(property "Footprint" "FRANK:Capacitor (0603, S)"
 			(at 47.9552 46.99 0)
 			(effects
@@
 			)
 		)
-		(property "Footprint" "FRANK:Resistor (0603)"
+		(property "Footprint" "FRANK:Resistor (0603, S)"
 			(at 246.38 131.318 90)
 			(effects
@@
 			)
 		)
-		(property "Footprint" "FRANK:Capacitor (0603)"
+		(property "Footprint" "FRANK:Capacitor (0603, S)"
 			(at 136.8552 46.99 0)
 			(effects
@@
 			)
 		)
-		(property "Footprint" "FRANK:Resistor (0603)"
+		(property "Footprint" "FRANK:Resistor (0603, S)"
 			(at 123.19 79.502 90)
 			(effects
@@
 			)
 		)
-		(property "Footprint" "FRANK:Resistor (0603)"
+		(property "Footprint" "FRANK:Resistor (0603, S)"
 			(at 123.19 71.882 90)
 			(effects
@@
 			)
 		)
-		(property "Footprint" "FRANK:Capacitor (0603)"
+		(property "Footprint" "FRANK:Capacitor (0603, S)"
 			(at 36.5252 46.99 0)
 			(effects
@@
 			)
 		)
-		(property "Footprint" "FRANK:Capacitor (0603)"
+		(property "Footprint" "FRANK:Capacitor (0603, S)"
 			(at 164.7952 125.73 0)
 			(effects
@@
 			)
 		)
-		(property "Footprint" "FRANK:Capacitor (0603)"
+		(property "Footprint" "FRANK:Capacitor (0603, S)"
 			(at 102.5652 46.99 0)
 			(effects
@@
 			)
 		)
-		(property "Footprint" "FRANK:Capacitor (0603)"
+		(property "Footprint" "FRANK:Capacitor (0603, S)"
 			(at 113.9952 46.99 0)
 			(effects
@@
 			)
 		)
-		(property "Footprint" "FRANK:Capacitor (0603)"
+		(property "Footprint" "FRANK:Capacitor (0603, S)"
 			(at 102.5652 62.23 0)
 			(effects
@@
 			)
 		)
-		(property "Footprint" "FRANK:Capacitor (0603)"
+		(property "Footprint" "FRANK:Capacitor (0603, S)"
 			(at 252.73 77.1652 0)
 			(effects
@@
 			)
 		)
-		(property "Footprint" "FRANK:Capacitor (0603)"
+		(property "Footprint" "FRANK:Capacitor (0603, S)"
 			(at 182.5752 46.99 0)
 			(effects
@@
 			)
 		)
-		(property "Footprint" "FRANK:Capacitor (0603)"
+		(property "Footprint" "FRANK:Capacitor (0603, S)"
 			(at 47.9552 62.23 0)
 			(effects
@@
 			)
 		)
-		(property "Footprint" "FRANK:Capacitor (0603)"
+		(property "Footprint" "FRANK:Capacitor (0603, S)"
 			(at 125.4252 46.99 0)
 			(effects
@@
 			)
 		)
-		(property "Footprint" "FRANK:Capacitor (0603)"
+		(property "Footprint" "FRANK:Capacitor (0603, S)"
 			(at 171.1452 46.99 0)
 			(effects
@@
 			)
 		)
-		(property "Footprint" "FRANK:Resistor (0603)"
+		(property "Footprint" "FRANK:Resistor (0603, S)"
 			(at 198.12 75.692 90)
 			(effects
@@
 			)
 		)
-		(property "Footprint" "FRANK:Capacitor (0603)"
+		(property "Footprint" "FRANK:Capacitor (0603, S)"
 			(at 148.2852 46.99 0)
 			(effects
@@
 			)
 		)
-		(property "Footprint" "FRANK:Capacitor (0603)"
+		(property "Footprint" "FRANK:Capacitor (0603, S)"
 			(at 159.7152 46.99 0)
 			(effects
