File: rs232.kicad_sch (KiCad schematic)
At the start: 22 parts, among them J3 TTL, J4 D-SUB 9 Male, Q1 2N7000, Q2 2N7000, Q3 2N7000, Q4 2N7000, U9 MAX232CSE+

Commit message: Cleanup WIP
Parts:
- renumbered C26 to C19, C27 to C20, C28 to C21, C29 to C22, R20 to R14, R21 to R15, R22 to R16, R23 to R17, R24 to R18, R25 to R19, U9 to U7
Changed lines of the file:
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@@
 		(on_board yes)
 		(dnp no)
-		(property "Reference" "R20"
+		(property "Reference" "R14"
 			(at 86.614 146.558 90)
 			(effects
@@
 			(project "protea"
 				(path "/8c0b3d8b-46d3-4173-ab1e-a61765f77d61/743e81f1-e5ae-4430-9dee-0c06cb416437"
-					(reference "R20")
+					(reference "R14")
 					(unit 1)
 				)
@@
 		(dnp no)
 		(fields_autoplaced yes)
-		(property "Reference" "C28"
+		(property "Reference" "C21"
 			(at 96.5263 92.71 90)
 			(effects
@@
 			(project "turbofrank"
 				(path "/8c0b3d8b-46d3-4173-ab1e-a61765f77d61/743e81f1-e5ae-4430-9dee-0c06cb416437"
-					(reference "C28")
+					(reference "C21")
 					(unit 1)
 				)
@@
 		(dnp no)
 		(fields_autoplaced yes)
-		(property "Reference" "#PWR063"
+		(property "Reference" "#PWR043"
 			(at 102.87 49.53 0)
 			(effects
@@
 			(project ""
 				(path "/8c0b3d8b-46d3-4173-ab1e-a61765f77d61/743e81f1-e5ae-4430-9dee-0c06cb416437"
-					(reference "#PWR063")
+					(reference "#PWR043")
 					(unit 1)
 				)
@@
 		(dnp no)
 		(fields_autoplaced yes)
-		(property "Reference" "C27"
+		(property "Reference" "C20"
 			(at 85.0963 97.79 90)
 			(effects
@@
 			(project "turbofrank"
 				(path "/8c0b3d8b-46d3-4173-ab1e-a61765f77d61/743e81f1-e5ae-4430-9dee-0c06cb416437"
-					(reference "C27")
+					(reference "C20")
 					(unit 1)
 				)
@@
 		(dnp no)
 		(fields_autoplaced yes)
-		(property "Reference" "C29"
+		(property "Reference" "C22"
 			(at 143.5163 81.28 90)
 			(effects
@@
 			(project ""
 				(path "/8c0b3d8b-46d3-4173-ab1e-a61765f77d61/743e81f1-e5ae-4430-9dee-0c06cb416437"
-					(reference "C29")
+					(reference "C22")
 					(unit 1)
 				)
@@
 		(dnp no)
 		(fields_autoplaced yes)
-		(property "Reference" "#PWR069"
+		(property "Reference" "#PWR049"
 			(at 156.21 49.53 0)
 			(effects
@@
 			(project "frank2"
 				(path "/8c0b3d8b-46d3-4173-ab1e-a61765f77d61/743e81f1-e5ae-4430-9dee-0c06cb416437"
-					(reference "#PWR069")
+					(reference "#PWR049")
 					(unit 1)
 				)
@@
 		(on_board yes)
 		(dnp no)
-		(property "Reference" "R24"
+		(property "Reference" "R18"
 			(at 154.94 54.61 90)
 			(effects
@@
 			(project "frank2"
 				(path "/8c0b3d8b-46d3-4173-ab1e-a61765f77d61/743e81f1-e5ae-4430-9dee-0c06cb416437"
-					(reference "R24")
+					(reference "R18")
 					(unit 1)
 				)
@@
 		(dnp no)
 		(fields_autoplaced yes)
-		(property "Reference" "#PWR073"
+		(property "Reference" "#PWR053"
 			(at 234.95 99.06 0)
 			(effects
@@
 			(project "protea"
 				(path "/8c0b3d8b-46d3-4173-ab1e-a61765f77d61/743e81f1-e5ae-4430-9dee-0c06cb416437"
-					(reference "#PWR073")
+					(reference "#PWR053")
 					(unit 1)
 				)
@@
 		(on_board yes)
 		(dnp no)
-		(property "Reference" "#PWR061"
+		(property "Reference" "#PWR041"
 			(at 88.9 173.99 0)
 			(effects
@@
 			(project "protea"
 				(path "/8c0b3d8b-46d3-4173-ab1e-a61765f77d61/743e81f1-e5ae-4430-9dee-0c06cb416437"
-					(reference "#PWR061")
+					(reference "#PWR041")
 					(unit 1)
 				)
@@
 		(on_board yes)
 		(dnp no)
-		(property "Reference" "C26"
+		(property "Reference" "C19"
 			(at 83.82 120.65 90)
 			(effects
@@
 			(project "turbofrank"
 				(path "/8c0b3d8b-46d3-4173-ab1e-a61765f77d61/743e81f1-e5ae-4430-9dee-0c06cb416437"
-					(reference "C26")
+					(reference "C19")
 					(unit 1)
 				)
@@
 		(dnp no)
 		(fields_autoplaced yes)
-		(property "Reference" "#PWR068"
+		(property "Reference" "#PWR048"
 			(at 153.67 85.09 0)
 			(effects
@@
 			(project "protea"
 				(path "/8c0b3d8b-46d3-4173-ab1e-a61765f77d61/743e81f1-e5ae-4430-9dee-0c06cb416437"
-					(reference "#PWR068")
+					(reference "#PWR048")
 					(unit 1)
 				)
@@
 		(on_board yes)
 		(dnp no)
-		(property "Reference" "#PWR065"
+		(property "Reference" "#PWR045"
 			(at 135.89 173.99 0)
 			(effects
@@
 			(project "protea"
 				(path "/8c0b3d8b-46d3-4173-ab1e-a61765f77d61/743e81f1-e5ae-4430-9dee-0c06cb416437"
-					(reference "#PWR065")
+					(reference "#PWR045")
 					(unit 1)
 				)
@@
 		(dnp no)
 		(fields_autoplaced yes)
-		(property "Reference" "#PWR070"
+		(property "Reference" "#PWR050"
 			(at 199.39 55.88 0)
 			(effects
@@
 			(project "frank2"
 				(path "/8c0b3d8b-46d3-4173-ab1e-a61765f77d61/743e81f1-e5ae-4430-9dee-0c06cb416437"
-					(reference "#PWR070")
+					(reference "#PWR050")
 					(unit 1)
 				)
@@
 		(on_board yes)
 		(dnp no)
-		(property "Reference" "R23"
+		(property "Reference" "R17"
 			(at 133.604 146.558 90)
 			(effects
@@
 			(project "protea"
 				(path "/8c0b3d8b-46d3-4173-ab1e-a61765f77d61/743e81f1-e5ae-4430-9dee-0c06cb416437"
-					(reference "R23")
+					(reference "R17")
 					(unit 1)
 				)
@@
 		(on_board yes)
 		(dnp no)
-		(property "Reference" "#PWR067"
+		(property "Reference" "#PWR047"
 			(at 152.4 166.37 0)
 			(effects
@@
 			(project "protea"
 				(path "/8c0b3d8b-46d3-4173-ab1e-a61765f77d61/743e81f1-e5ae-4430-9dee-0c06cb416437"
-					(reference "#PWR067")
+					(reference "#PWR047")
 					(unit 1)
 				)
@@
 		(dnp no)
 		(fields_autoplaced yes)
-		(property "Reference" "#PWR064"
+		(property "Reference" "#PWR044"
 			(at 135.89 144.78 0)
 			(effects
@@
 			(project "protea"
 				(path "/8c0b3d8b-46d3-4173-ab1e-a61765f77d61/743e81f1-e5ae-4430-9dee-0c06cb416437"
-					(reference "#PWR064")
+					(reference "#PWR044")
 					(unit 1)
 				)
@@
 		(dnp no)
 		(fields_autoplaced yes)
-		(property "Reference" "U9"
+		(property "Reference" "U7"
 			(at 133.35 91.44 0)
 			(effects
@@
 			(project "frank2"
 				(path "/8c0b3d8b-46d3-4173-ab1e-a61765f77d61/743e81f1-e5ae-4430-9dee-0c06cb416437"
-					(reference "U9")
+					(reference "U7")
 					(unit 1)
 				)
@@
 		(dnp no)
 		(fields_autoplaced yes)
-		(property "Reference" "#PWR059"
+		(property "Reference" "#PWR039"
 			(at 69.85 114.3 0)
 			(effects
@@
 			(project "frank2"
 				(path "/8c0b3d8b-46d3-4173-ab1e-a61765f77d61/743e81f1-e5ae-4430-9dee-0c06cb416437"
-					(reference "#PWR059")
+					(reference "#PWR039")
 					(unit 1)
 				)
@@
 		(on_board yes)
 		(dnp no)
-		(property "Reference" "#PWR071"
+		(property "Reference" "#PWR051"
 			(at 212.09 90.17 0)
 			(effects
@@
 			(project "protea"
 				(path "/8c0b3d8b-46d3-4173-ab1e-a61765f77d61/743e81f1-e5ae-4430-9dee-0c06cb416437"
-					(reference "#PWR071")
+					(reference "#PWR051")
 					(unit 1)
 				)
@@
 		(on_board yes)
 		(dnp no)
-		(property "Reference" "R21"
+		(property "Reference" "R15"
 			(at 101.6 54.61 90)
 			(effects
@@
 			(project "frank2"
 				(path "/8c0b3d8b-46d3-4173-ab1e-a61765f77d61/743e81f1-e5ae-4430-9dee-0c06cb416437"
-					(reference "R21")
+					(reference "R15")
 					(unit 1)
 				)
@@
 		(on_board yes)
 		(dnp no)
-		(property "Reference" "#PWR066"
+		(property "Reference" "#PWR046"
 			(at 154.94 101.6 0)
 			(effects
@@
 			(project "frank2"
 				(path "/8c0b3d8b-46d3-4173-ab1e-a61765f77d61/743e81f1-e5ae-4430-9dee-0c06cb416437"
-					(reference "#PWR066")
+					(reference "#PWR046")
 					(unit 1)
 				)
@@
 		(dnp no)
 		(fields_autoplaced yes)
-		(property "Reference" "#PWR072"
+		(property "Reference" "#PWR052"
 			(at 234.95 93.98 0)
 			(effects
@@
 			(project "protea"
 				(path "/8c0b3d8b-46d3-4173-ab1e-a61765f77d61/743e81f1-e5ae-4430-9dee-0c06cb416437"
-					(reference "#PWR072")
+					(reference "#PWR052")
 					(unit 1)
 				)
@@
 		(on_board yes)
 		(dnp no)
-		(property "Reference" "R25"
+		(property "Reference" "R19"
 			(at 150.114 140.208 90)
 			(effects
@@
 			(project "protea"
 				(path "/8c0b3d8b-46d3-4173-ab1e-a61765f77d61/743e81f1-e5ae-4430-9dee-0c06cb416437"
-					(reference "R25")
+					(reference "R19")
 					(unit 1)
 				)
@@
 		(dnp no)
 		(fields_autoplaced yes)
-		(property "Reference" "#PWR060"
+		(property "Reference" "#PWR040"
 			(at 88.9 144.78 0)
 			(effects
@@
 			(project "protea"
 				(path "/8c0b3d8b-46d3-4173-ab1e-a61765f77d61/743e81f1-e5ae-4430-9dee-0c06cb416437"
-					(reference "#PWR060")
+					(reference "#PWR040")
 					(unit 1)
 				)
@@
 		(on_board yes)
 		(dnp no)
-		(property "Reference" "#PWR062"
+		(property "Reference" "#PWR042"
 			(at 105.41 166.37 0)
 			(effects
@@
 			(project "protea"
 				(path "/8c0b3d8b-46d3-4173-ab1e-a61765f77d61/743e81f1-e5ae-4430-9dee-0c06cb416437"
-					(reference "#PWR062")
+					(reference "#PWR042")
 					(unit 1)
 				)
@@
 		(on_board yes)
 		(dnp no)
-		(property "Reference" "R22"
+		(property "Reference" "R16"
 			(at 103.124 140.208 90)
 			(effects
@@
 			(project "protea"
 				(path "/8c0b3d8b-46d3-4173-ab1e-a61765f77d61/743e81f1-e5ae-4430-9dee-0c06cb416437"
-					(reference "R22")
-					(unit 1)
-				)
+					(reference "R16")
+					(unit 1)
+				)

Commit message: HW 1.01
Parts:
- C19, C20, C21, C22: footprint FRANK:Capacitor (0603, S) -> FRANK:Capacitor (0603)
- R14, R15, R16, R17, R18, R19: footprint FRANK:Resistor (0603, S) -> FRANK:Resistor (0603)
Changed lines of the file:
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@@
 		(rev "${VERSION}")
 		(company "Mikhail Matveev")
-		(comment 1 "https://github.com/xtremespb/frank")
+		(comment 1 "https://github.com/rh1tech/protea")
 	)
 	(junction
@@
 			)
 		)
-		(property "Footprint" "FRANK:Resistor (0603, S)"
+		(property "Footprint" "FRANK:Resistor (0603)"
 			(at 90.678 144.78 90)
 			(effects
@@
 			)
 		)
-		(property "Footprint" "FRANK:Capacitor (0603, S)"
+		(property "Footprint" "FRANK:Capacitor (0603)"
 			(at 96.52 99.06 0)
 			(effects
@@
 			)
 		)
-		(property "Footprint" "FRANK:Capacitor (0603, S)"
+		(property "Footprint" "FRANK:Capacitor (0603)"
 			(at 85.09 104.14 0)
 			(effects
@@
 			)
 		)
-		(property "Footprint" "FRANK:Capacitor (0603, S)"
+		(property "Footprint" "FRANK:Capacitor (0603)"
 			(at 143.51 87.63 0)
 			(effects
@@
 			)
 		)
-		(property "Footprint" "FRANK:Resistor (0603, S)"
+		(property "Footprint" "FRANK:Resistor (0603)"
 			(at 154.178 54.61 90)
 			(effects
@@
 			)
 		)
-		(property "Footprint" "FRANK:Capacitor (0603, S)"
+		(property "Footprint" "FRANK:Capacitor (0603)"
 			(at 83.82 114.3 0)
 			(effects
@@
 			)
 		)
-		(property "Footprint" "FRANK:Resistor (0603, S)"
+		(property "Footprint" "FRANK:Resistor (0603)"
 			(at 137.668 144.78 90)
 			(effects
@@
 			)
 		)
-		(property "Footprint" "FRANK:Resistor (0603, S)"
+		(property "Footprint" "FRANK:Resistor (0603)"
 			(at 100.838 54.61 90)
 			(effects
@@
 			)
 		)
-		(property "Footprint" "FRANK:Resistor (0603, S)"
+		(property "Footprint" "FRANK:Resistor (0603)"
 			(at 154.178 138.43 90)
 			(effects
@@
 			)
 		)
-		(property "Footprint" "FRANK:Resistor (0603, S)"
+		(property "Footprint" "FRANK:Resistor (0603)"
 			(at 107.188 138.43 90)
 			(effects

Commit message: HW 1.01
Parts:
- C19, C20, C21, C22: footprint FRANK:Capacitor (0603) -> FRANK:Capacitor (0603, S)
- R14, R15, R16, R17, R18, R19: footprint FRANK:Resistor (0603) -> FRANK:Resistor (0603, S)
Changed lines of the file:
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@@
 			)
 		)
-		(property "Footprint" "FRANK:Resistor (0603)"
+		(property "Footprint" "FRANK:Resistor (0603, S)"
 			(at 90.678 144.78 90)
 			(effects
@@
 			)
 		)
-		(property "Footprint" "FRANK:Capacitor (0603)"
+		(property "Footprint" "FRANK:Capacitor (0603, S)"
 			(at 96.52 99.06 0)
 			(effects
@@
 			)
 		)
-		(property "Footprint" "FRANK:Capacitor (0603)"
+		(property "Footprint" "FRANK:Capacitor (0603, S)"
 			(at 85.09 104.14 0)
 			(effects
@@
 			)
 		)
-		(property "Footprint" "FRANK:Capacitor (0603)"
+		(property "Footprint" "FRANK:Capacitor (0603, S)"
 			(at 143.51 87.63 0)
 			(effects
@@
 			)
 		)
-		(property "Footprint" "FRANK:Resistor (0603)"
+		(property "Footprint" "FRANK:Resistor (0603, S)"
 			(at 154.178 54.61 90)
 			(effects
@@
 			)
 		)
-		(property "Footprint" "FRANK:Capacitor (0603)"
+		(property "Footprint" "FRANK:Capacitor (0603, S)"
 			(at 83.82 114.3 0)
 			(effects
@@
 			)
 		)
-		(property "Footprint" "FRANK:Resistor (0603)"
+		(property "Footprint" "FRANK:Resistor (0603, S)"
 			(at 137.668 144.78 90)
 			(effects
@@
 			)
 		)
-		(property "Footprint" "FRANK:Resistor (0603)"
+		(property "Footprint" "FRANK:Resistor (0603, S)"
 			(at 100.838 54.61 90)
 			(effects
@@
 			)
 		)
-		(property "Footprint" "FRANK:Resistor (0603)"
+		(property "Footprint" "FRANK:Resistor (0603, S)"
 			(at 154.178 138.43 90)
 			(effects
@@
 			)
 		)
-		(property "Footprint" "FRANK:Resistor (0603)"
+		(property "Footprint" "FRANK:Resistor (0603, S)"
 			(at 107.188 138.43 90)
 			(effects
