File: sd.kicad_sch (KiCad schematic)
At the start: 5 parts, among them J5 0475710001

Commit message: Cleanup WIP
Parts:
- renumbered C33 to C26, R30 to R24, R31 to R25, R32 to R26
Changed lines of the file:
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@@
 		(on_board yes)
 		(dnp no)
-		(property "Reference" "R30"
+		(property "Reference" "R24"
 			(at 125.222 114.3 90)
 			(effects
@@
 			(project "protea32"
 				(path "/8c0b3d8b-46d3-4173-ab1e-a61765f77d61/dcad9fa4-633b-4c75-add1-11aea46e0585"
-					(reference "R30")
+					(reference "R24")
 					(unit 1)
 				)
@@
 		(on_board yes)
 		(dnp no)
-		(property "Reference" "C33"
+		(property "Reference" "C26"
 			(at 194.2084 98.171 0)
 			(effects
@@
 			(project "minifrank_rm1"
 				(path "/8c0b3d8b-46d3-4173-ab1e-a61765f77d61/dcad9fa4-633b-4c75-add1-11aea46e0585"
-					(reference "C33")
+					(reference "C26")
 					(unit 1)
 				)
@@
 		(dnp no)
 		(fields_autoplaced yes)
-		(property "Reference" "#PWR0108"
+		(property "Reference" "#PWR088"
 			(at 184.15 91.44 0)
 			(effects
@@
 			(project "minifrank_rm1"
 				(path "/8c0b3d8b-46d3-4173-ab1e-a61765f77d61/dcad9fa4-633b-4c75-add1-11aea46e0585"
-					(reference "#PWR0108")
+					(reference "#PWR088")
 					(unit 1)
 				)
@@
 		(on_board yes)
 		(dnp no)
-		(property "Reference" "#PWR0109"
+		(property "Reference" "#PWR089"
 			(at 203.2 95.25 0)
 			(effects
@@
 			(project "minifrank_rm1"
 				(path "/8c0b3d8b-46d3-4173-ab1e-a61765f77d61/dcad9fa4-633b-4c75-add1-11aea46e0585"
-					(reference "#PWR0109")
+					(reference "#PWR089")
 					(unit 1)
 				)
@@
 		(dnp no)
 		(fields_autoplaced yes)
-		(property "Reference" "#PWR0103"
+		(property "Reference" "#PWR083"
 			(at 120.65 95.25 0)
 			(effects
@@
 			(project "minifrank_rm1"
 				(path "/8c0b3d8b-46d3-4173-ab1e-a61765f77d61/dcad9fa4-633b-4c75-add1-11aea46e0585"
-					(reference "#PWR0103")
+					(reference "#PWR083")
 					(unit 1)
 				)
@@
 		(on_board yes)
 		(dnp no)
-		(property "Reference" "R32"
+		(property "Reference" "R26"
 			(at 167.132 109.22 90)
 			(effects
@@
 			(project "protea32"
 				(path "/8c0b3d8b-46d3-4173-ab1e-a61765f77d61/dcad9fa4-633b-4c75-add1-11aea46e0585"
-					(reference "R32")
+					(reference "R26")
 					(unit 1)
 				)
@@
 		(on_board yes)
 		(dnp no)
-		(property "Reference" "R31"
+		(property "Reference" "R25"
 			(at 163.068 86.36 90)
 			(effects
@@
 			(project "protea32"
 				(path "/8c0b3d8b-46d3-4173-ab1e-a61765f77d61/dcad9fa4-633b-4c75-add1-11aea46e0585"
-					(reference "R31")
+					(reference "R25")
 					(unit 1)
 				)
@@
 		(on_board yes)
 		(dnp no)
-		(property "Reference" "#PWR0101"
+		(property "Reference" "#PWR081"
 			(at 123.19 114.3 0)
 			(effects
@@
 			(project "protea32"
 				(path "/8c0b3d8b-46d3-4173-ab1e-a61765f77d61/dcad9fa4-633b-4c75-add1-11aea46e0585"
-					(reference "#PWR0101")
+					(reference "#PWR081")
 					(unit 1)
 				)
@@
 		(dnp no)
 		(fields_autoplaced yes)
-		(property "Reference" "#PWR0105"
+		(property "Reference" "#PWR085"
 			(at 166.37 100.33 0)
 			(effects
@@
 			(project "minifrank_rm1"
 				(path "/8c0b3d8b-46d3-4173-ab1e-a61765f77d61/dcad9fa4-633b-4c75-add1-11aea46e0585"
-					(reference "#PWR0105")
+					(reference "#PWR085")
 					(unit 1)
 				)
@@
 		(on_board yes)
 		(dnp no)
-		(property "Reference" "#PWR0106"
+		(property "Reference" "#PWR086"
 			(at 165.1 86.36 0)
 			(effects
@@
 			(project "protea32"
 				(path "/8c0b3d8b-46d3-4173-ab1e-a61765f77d61/dcad9fa4-633b-4c75-add1-11aea46e0585"
-					(reference "#PWR0106")
+					(reference "#PWR086")
 					(unit 1)
 				)
@@
 		(dnp no)
 		(fields_autoplaced yes)
-		(property "Reference" "#PWR0104"
+		(property "Reference" "#PWR084"
 			(at 120.65 97.79 0)
 			(effects
@@
 			(project "minifrank_rm1"
 				(path "/8c0b3d8b-46d3-4173-ab1e-a61765f77d61/dcad9fa4-633b-4c75-add1-11aea46e0585"
-					(reference "#PWR0104")
+					(reference "#PWR084")
 					(unit 1)
 				)
@@
 		(dnp no)
 		(fields_autoplaced yes)
-		(property "Reference" "#PWR0102"
+		(property "Reference" "#PWR082"
 			(at 120.65 92.71 0)
 			(effects
@@
 			(project "minifrank_rm1"
 				(path "/8c0b3d8b-46d3-4173-ab1e-a61765f77d61/dcad9fa4-633b-4c75-add1-11aea46e0585"
-					(reference "#PWR0102")
+					(reference "#PWR082")
 					(unit 1)
 				)
@@
 		(on_board yes)
 		(dnp no)
-		(property "Reference" "#PWR0107"
+		(property "Reference" "#PWR087"
 			(at 165.1 109.22 0)
 			(effects
@@
 			(project "protea32"
 				(path "/8c0b3d8b-46d3-4173-ab1e-a61765f77d61/dcad9fa4-633b-4c75-add1-11aea46e0585"
-					(reference "#PWR0107")
-					(unit 1)
-				)
+					(reference "#PWR087")
+					(unit 1)
+				)

Commit message: HW 1.01
Parts:
- added R27: 10K, FRANK:Resistor (0603), symbol Protea:R
- C26: footprint FRANK:Capacitor (0603, S) -> FRANK:Capacitor (0603)
- R24, R25, R26: footprint FRANK:Resistor (0603, S) -> FRANK:Resistor (0603)
Connections:
- net +3V3: now also R27.2
- net CLK: now also R25.1
- net CMD: now also R27.1; no longer R25.1

Commit message: HW 1.01
Parts:
- C26: footprint FRANK:Capacitor (0603) -> FRANK:Capacitor (0603, S)
- R24, R25, R26, R27: footprint FRANK:Resistor (0603) -> FRANK:Resistor (0603, S)
Changed lines of the file:
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@@
 			)
 		)
-		(property "Footprint" "FRANK:Resistor (0603)"
+		(property "Footprint" "FRANK:Resistor (0603, S)"
 			(at 120.142 118.11 90)
 			(effects
@@
 			)
 		)
-		(property "Footprint" "FRANK:Capacitor (0603)"
+		(property "Footprint" "FRANK:Capacitor (0603, S)"
 			(at 189.23 96.2152 0)
 			(effects
@@
 			)
 		)
-		(property "Footprint" "FRANK:Resistor (0603)"
+		(property "Footprint" "FRANK:Resistor (0603, S)"
 			(at 164.338 82.55 90)
 			(effects
@@
 			)
 		)
-		(property "Footprint" "FRANK:Resistor (0603)"
+		(property "Footprint" "FRANK:Resistor (0603, S)"
 			(at 163.322 113.03 90)
 			(effects
@@
 			)
 		)
-		(property "Footprint" "FRANK:Resistor (0603)"
+		(property "Footprint" "FRANK:Resistor (0603, S)"
 			(at 171.958 82.55 90)
 			(effects
