File: usb2ttl.kicad_sch (KiCad schematic)
At the start: 6 parts, among them U14 CH340C

Commit message: Cleanup WIP
Parts:
- renumbered C54 to C47, R45 to R39, R46 to R40, U14 to U13
Changed lines of the file:
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@@
 		(on_board yes)
 		(dnp no)
-		(property "Reference" "U14"
+		(property "Reference" "U13"
 			(at 140.97 70.866 0)
 			(effects
@@
 			(project "echo"
 				(path "/8c0b3d8b-46d3-4173-ab1e-a61765f77d61/1802e340-067b-4c70-8138-d845438ae144"
-					(reference "U14")
+					(reference "U13")
 					(unit 1)
 				)
@@
 		(on_board yes)
 		(dnp no)
-		(property "Reference" "R46"
+		(property "Reference" "R40"
 			(at 195.834 82.55 90)
 			(effects
@@
 			(project "echo"
 				(path "/8c0b3d8b-46d3-4173-ab1e-a61765f77d61/1802e340-067b-4c70-8138-d845438ae144"
-					(reference "R46")
+					(reference "R40")
 					(unit 1)
 				)
@@
 		(on_board yes)
 		(dnp no)
-		(property "Reference" "#PWR0155"
+		(property "Reference" "#PWR0135"
 			(at 196.85 74.93 0)
 			(effects
@@
 			(project ""
 				(path "/8c0b3d8b-46d3-4173-ab1e-a61765f77d61/1802e340-067b-4c70-8138-d845438ae144"
-					(reference "#PWR0155")
+					(reference "#PWR0135")
 					(unit 1)
 				)
@@
 		(on_board yes)
 		(dnp no)
-		(property "Reference" "#PWR0153"
+		(property "Reference" "#PWR0133"
 			(at 119.38 82.55 0)
 			(effects
@@
 			(project "protea"
 				(path "/8c0b3d8b-46d3-4173-ab1e-a61765f77d61/1802e340-067b-4c70-8138-d845438ae144"
-					(reference "#PWR0153")
+					(reference "#PWR0133")
 					(unit 1)
 				)
@@
 		(on_board yes)
 		(dnp no)
-		(property "Reference" "R45"
+		(property "Reference" "R39"
 			(at 185.42 82.55 90)
 			(effects
@@
 			(project "echo"
 				(path "/8c0b3d8b-46d3-4173-ab1e-a61765f77d61/1802e340-067b-4c70-8138-d845438ae144"
-					(reference "R45")
+					(reference "R39")
 					(unit 1)
 				)
@@
 		(dnp no)
 		(fields_autoplaced yes)
-		(property "Reference" "#PWR0152"
+		(property "Reference" "#PWR0132"
 			(at 109.22 74.93 0)
 			(effects
@@
 			(project ""
 				(path "/8c0b3d8b-46d3-4173-ab1e-a61765f77d61/1802e340-067b-4c70-8138-d845438ae144"
-					(reference "#PWR0152")
+					(reference "#PWR0132")
 					(unit 1)
 				)
@@
 		(on_board yes)
 		(dnp no)
-		(property "Reference" "#PWR0154"
+		(property "Reference" "#PWR0134"
 			(at 171.45 92.71 0)
 			(effects
@@
 			(project "echo"
 				(path "/8c0b3d8b-46d3-4173-ab1e-a61765f77d61/1802e340-067b-4c70-8138-d845438ae144"
-					(reference "#PWR0154")
+					(reference "#PWR0134")
 					(unit 1)
 				)
@@
 		(on_board yes)
 		(dnp no)
-		(property "Reference" "C54"
+		(property "Reference" "C47"
 			(at 171.958 78.74 0)
 			(effects
@@
 			(project "echo"
 				(path "/8c0b3d8b-46d3-4173-ab1e-a61765f77d61/1802e340-067b-4c70-8138-d845438ae144"
-					(reference "C54")
-					(unit 1)
-				)
+					(reference "C47")
+					(unit 1)
+				)

Commit message: HW 1.01
Parts:
- C29: renamed from C47; footprint FRANK:Capacitor (0603, S) -> FRANK:Capacitor (0603)
- R32: renamed from R39; footprint FRANK:Resistor (0603, S) -> FRANK:Resistor (0603)
- R33: renamed from R40; footprint FRANK:Resistor (0603, S) -> FRANK:Resistor (0603)
- renumbered LD5 to LD4, LD6 to LD5
Changed lines of the file:
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@@
 		(rev "${VERSION}")
 		(company "Mikhail Matveev")
-		(comment 1 "https://github.com/xtremespb/frank")
+		(comment 1 "https://github.com/rh1tech/protea")
 	)
 	(junction
@@
 		(on_board yes)
 		(dnp no)
-		(property "Reference" "LD5"
+		(property "Reference" "LD4"
 			(at 179.832 91.694 0)
 			(effects
@@
 			(project "echo"
 				(path "/8c0b3d8b-46d3-4173-ab1e-a61765f77d61/1802e340-067b-4c70-8138-d845438ae144"
-					(reference "LD5")
+					(reference "LD4")
 					(unit 1)
 				)
@@
 		(on_board yes)
 		(dnp no)
-		(property "Reference" "R40"
+		(property "Reference" "R33"
 			(at 195.834 82.55 90)
 			(effects
@@
 			)
 		)
-		(property "Footprint" "FRANK:Resistor (0603, S)"
+		(property "Footprint" "FRANK:Resistor (0603)"
 			(at 193.04 82.55 0)
 			(effects
@@
 			(project "echo"
 				(path "/8c0b3d8b-46d3-4173-ab1e-a61765f77d61/1802e340-067b-4c70-8138-d845438ae144"
-					(reference "R40")
+					(reference "R33")
 					(unit 1)
 				)
@@
 		(on_board yes)
 		(dnp no)
-		(property "Reference" "#PWR0135"
+		(property "Reference" "#PWR0110"
 			(at 196.85 74.93 0)
 			(effects
@@
 			(project ""
 				(path "/8c0b3d8b-46d3-4173-ab1e-a61765f77d61/1802e340-067b-4c70-8138-d845438ae144"
-					(reference "#PWR0135")
+					(reference "#PWR0110")
 					(unit 1)
 				)
@@
 		(on_board yes)
 		(dnp no)
-		(property "Reference" "#PWR0133"
+		(property "Reference" "#PWR0108"
 			(at 119.38 82.55 0)
 			(effects
@@
 			(project "protea"
 				(path "/8c0b3d8b-46d3-4173-ab1e-a61765f77d61/1802e340-067b-4c70-8138-d845438ae144"
-					(reference "#PWR0133")
+					(reference "#PWR0108")
 					(unit 1)
 				)
@@
 		(on_board yes)
 		(dnp no)
-		(property "Reference" "R39"
+		(property "Reference" "R32"
 			(at 185.42 82.55 90)
 			(effects
@@
 			)
 		)
-		(property "Footprint" "FRANK:Resistor (0603, S)"
+		(property "Footprint" "FRANK:Resistor (0603)"
 			(at 182.88 82.55 0)
 			(effects
@@
 			(project "echo"
 				(path "/8c0b3d8b-46d3-4173-ab1e-a61765f77d61/1802e340-067b-4c70-8138-d845438ae144"
-					(reference "R39")
+					(reference "R32")
 					(unit 1)
 				)
@@
 		(dnp no)
 		(fields_autoplaced yes)
-		(property "Reference" "#PWR0132"
+		(property "Reference" "#PWR0107"
 			(at 109.22 74.93 0)
 			(effects
@@
 			(project ""
 				(path "/8c0b3d8b-46d3-4173-ab1e-a61765f77d61/1802e340-067b-4c70-8138-d845438ae144"
-					(reference "#PWR0132")
+					(reference "#PWR0107")
 					(unit 1)
 				)
@@
 		(on_board yes)
 		(dnp no)
-		(property "Reference" "#PWR0134"
+		(property "Reference" "#PWR0109"
 			(at 171.45 92.71 0)
 			(effects
@@
 			(project "echo"
 				(path "/8c0b3d8b-46d3-4173-ab1e-a61765f77d61/1802e340-067b-4c70-8138-d845438ae144"
-					(reference "#PWR0134")
+					(reference "#PWR0109")
 					(unit 1)
 				)
@@
 		(on_board yes)
 		(dnp no)
-		(property "Reference" "LD6"
+		(property "Reference" "LD5"
 			(at 189.992 91.694 0)
 			(effects
@@
 			(project "echo"
 				(path "/8c0b3d8b-46d3-4173-ab1e-a61765f77d61/1802e340-067b-4c70-8138-d845438ae144"
-					(reference "LD6")
+					(reference "LD5")
 					(unit 1)
 				)
@@
 		(on_board yes)
 		(dnp no)
-		(property "Reference" "C47"
+		(property "Reference" "C29"
 			(at 171.958 78.74 0)
 			(effects
@@
 			)
 		)
-		(property "Footprint" "FRANK:Capacitor (0603, S)"
+		(property "Footprint" "FRANK:Capacitor (0603)"
 			(at 171.45 81.28 0)
 			(effects
@@
 			(project "echo"
 				(path "/8c0b3d8b-46d3-4173-ab1e-a61765f77d61/1802e340-067b-4c70-8138-d845438ae144"
-					(reference "C47")
+					(reference "C29")
 					(unit 1)
 				)

Commit message: HW 1.01
Parts:
- C29: footprint FRANK:Capacitor (0603) -> FRANK:Capacitor (0603, S)
- R32, R33: footprint FRANK:Resistor (0603) -> FRANK:Resistor (0603, S)
Changed lines of the file:
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@@
 			)
 		)
-		(property "Footprint" "FRANK:Resistor (0603)"
+		(property "Footprint" "FRANK:Resistor (0603, S)"
 			(at 193.04 82.55 0)
 			(effects
@@
 			)
 		)
-		(property "Footprint" "FRANK:Resistor (0603)"
+		(property "Footprint" "FRANK:Resistor (0603, S)"
 			(at 182.88 82.55 0)
 			(effects
@@
 			)
 		)
-		(property "Footprint" "FRANK:Capacitor (0603)"
+		(property "Footprint" "FRANK:Capacitor (0603, S)"
 			(at 171.45 81.28 0)
 			(effects
