File: esp32-d0wd-v3.kicad_sch (KiCad schematic)
At the start: 34 parts, among them IC1 ESP32-D0WD-V3, Q6 UMH3N, Y3 40MHz

Commit message: Cleanup WIP
Parts:
- renumbered AE2 to AE1, C34 to C27, C35 to C28, C36 to C29, C37 to C30, C38 to C31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

Commit message: HW 1.01
Parts:
- removed LD4: Blue, FRANK:LED (0805), symbol Protea:LED_Small
- removed R37: 5.1K, FRANK:Resistor (0603, S), symbol Protea:R_Small
- renumbered C27 to C30, C28 to C31, C29 to C32, C30 to C33, C31 to C34, C32 to C35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
